Commit message: update_code 28

File: urdf/model.urdf (robot description, URDF)
Before this commit: robot jmbot, 8 links, 7 joints
Links:
- link UNION: geometry collision mesh filename=package://jmbot/urdf/meshes/UNION_bueno.stl; visual mesh filename=package://jmbot/urdf/meshes/UNION_bueno.obj
- link brazomedio: geometry collision mesh filename=package://jmbot/urdf/meshes/brazomedio_bueno.stl; visual mesh filename=package://jmbot/urdf/meshes/brazomedio_bueno.obj
- link pinza: geometry collision mesh filename=package://jmbot/urdf/meshes/Pinza_base_bueno.stl; visual mesh filename=package://jmbot/urdf/meshes/Pinza_base_bueno.obj
- link pinza_extremo: geometry collision mesh filename=package://jmbot/urdf/meshes/Pinza_bueno.stl; visual mesh filename=package://jmbot/urdf/meshes/Pinza_bueno.obj
